File: hardware_v3/pi-parport.sch (KiCad schematic (older format))
At the start: 14 parts, among them J1 CONN_01X02, J2 40HAT, J3 Conn_02x13_Odd_Even, U1 CAT24C32, U2 SN74LVC161284DLR

Commit message: hardware_v3: add BOM manufacturer part numbers
Parts:
- J1: Digi-Key_PN (none) -> 952-2262-ND; MPN (none) -> M20-9990246; Manufacturer (none) -> Harwin Inc.
- J2: Digi-Key_PN (none) -> S5750-20-ND; MPN (none) -> NPPN202AFCN-RC; Manufacturer (none) -> Sullins Connector Solutions
- J3: Digi-Key_PN (none) -> 23-0877602616-ND; MPN (none) -> 0877602616; Manufacturer (none) -> Molex
- R2: Digi-Key_PN (none) -> P10.0KCCT-ND; MPN (none) -> ERJ-6ENF1002V; Manufacturer (none) -> Panasonic Electronic Components
- R3, R4: Digi-Key_PN (none) -> P3.90KCCT-ND; MPN (none) -> ERJ-6ENF3901V; Manufacturer (none) -> Panasonic Electronic Components
- R5: Digi-Key_PN (none) -> P1.40KCCT-ND; MPN (none) -> ERJ-6ENF1401V; Manufacturer (none) -> Panasonic Electronic Components
- U1: Digi-Key_PN (none) -> CAT24C32WI-GT3CT-ND; MPN (none) -> CAT24C32WI-GT3; Manufacturer (none) -> ON Semiconductor
- U2: Digi-Key_PN (none) -> 296-8467-1-ND; MPN (none) -> SN74LVC161284DLR; Manufacturer (none) -> Texas Instruments
Changed lines of the file:
@@
 EESchema Schematic File Version 4
+LIBS:pi-parport-cache
 EELAYER 30 0
 EELAYER END
@@
 F 2 "Connector_PinSocket_2.54mm:PinSocket_2x20_P2.54mm_Vertical" H 2400 2200 50  0001 C CNN
 F 3 "" H 1700 2000 50  0000 C CNN
+F 4 "S5750-20-ND" H 2400 2000 50  0001 C CNN "Digi-Key_PN"
+F 5 "NPPN202AFCN-RC" H 2400 2000 50  0001 C CNN "MPN"
+F 6 "Sullins Connector Solutions" H 2400 2000 50  0001 C CNN "Manufacturer"
 	1    2400 2000
 	1    0    0    -1
@@
 F 1 "CAT24C32" H 2800 6300 50  0000 C CNN
 F 2 "Package_SO:SO-8_3.9x4.9mm_P1.27mm" H 3050 5950 50  0001 C CNN
-F 3 "" H 3050 5950 50  0000 C CNN
+F 3 "https://www.onsemi.com/pub/Collateral/CAT24C32-D.PDF" H 3050 5950 50  0001 C CNN
+F 4 "CAT24C32WI-GT3CT-ND" H 3050 5950 50  0001 C CNN "Digi-Key_PN"
+F 5 "CAT24C32WI-GT3" H 3050 5950 50  0001 C CNN "MPN"
+F 6 "ON Semiconductor" H 3050 5950 50  0001 C CNN "Manufacturer"
 	1    3050 5950
 	1    0    0    -1
@@
 F 2 "Resistor_SMD:R_0805_2012Metric_Pad1.15x1.40mm_HandSolder" V 3630 5700 50  0001 C CNN
 F 3 "" H 3700 5700 50  0001 C CNN
+F 4 "P3.90KCCT-ND" V 3700 5700 50  0001 C CNN "Digi-Key_PN"
+F 5 "ERJ-6ENF3901V" V 3700 5700 50  0001 C CNN "MPN"
+F 6 "Panasonic Electronic Components" V 3700 5700 50  0001 C CNN "Manufacturer"
 	1    3700 5700
 	1    0    0    -1
@@
 F 2 "Resistor_SMD:R_0805_2012Metric_Pad1.15x1.40mm_HandSolder" V 3830 5700 50  0001 C CNN
 F 3 "" H 3900 5700 50  0001 C CNN
+F 4 "P3.90KCCT-ND" V 3900 5700 50  0001 C CNN "Digi-Key_PN"
+F 5 "ERJ-6ENF3901V" V 3900 5700 50  0001 C CNN "MPN"
+F 6 "Panasonic Electronic Components" V 3900 5700 50  0001 C CNN "Manufacturer"
 	1    3900 5700
 	1    0    0    -1
@@
 F 2 "Connector_PinHeader_2.54mm:PinHeader_1x02_P2.54mm_Vertical" H 1500 6200 50  0001 C CNN
 F 3 "" H 1500 6200 50  0000 C CNN
+F 4 "952-2262-ND" H 1500 6200 50  0001 C CNN "Digi-Key_PN"
+F 5 "M20-9990246" H 1500 6200 50  0001 C CNN "MPN"
+F 6 "Harwin Inc." H 1500 6200 50  0001 C CNN "Manufacturer"
 	1    1500 6200
 	-1   0    0    1
@@
 F 2 "Resistor_SMD:R_0805_2012Metric_Pad1.15x1.40mm_HandSolder" V 1780 5700 50  0001 C CNN
 F 3 "" H 1850 5700 50  0001 C CNN
+F 4 "P10.0KCCT-ND" V 1850 5700 50  0001 C CNN "Digi-Key_PN"
+F 5 "ERJ-6ENF1002V" V 1850 5700 50  0001 C CNN "MPN"
+F 6 "Panasonic Electronic Components" V 1850 5700 50  0001 C CNN "Manufacturer"
 	1    1850 5700
 	-1   0    0    1
@@
 F 2 "Package_SO:SSOP-48_7.5x15.9mm_P0.635mm" H 6700 3000 60  0001 C CNN
 F 3 "http://www.ti.com/lit/ds/symlink/sn74lvc161284.pdf" H 5975 3681 60  0001 C CNN
+F 4 "296-8467-1-ND" H 7800 2550 50  0001 C CNN "Digi-Key_PN"
+F 5 "SN74LVC161284DLR" H 7800 2550 50  0001 C CNN "MPN"
+F 6 "Texas Instruments" H 7800 2550 50  0001 C CNN "Manufacturer"
 	1    7800 2550
 	1    0    0    -1
@@
 F 2 "Resistor_SMD:R_0805_2012Metric_Pad1.15x1.40mm_HandSolder" V 6680 3300 50  0001 C CNN
 F 3 "" H 6750 3300 50  0001 C CNN
+F 4 "P1.40KCCT-ND" V 6750 3300 50  0001 C CNN "Digi-Key_PN"
+F 5 "ERJ-6ENF1401V" V 6750 3300 50  0001 C CNN "MPN"
+F 6 "Panasonic Electronic Components" V 6750 3300 50  0001 C CNN "Manufacturer"
 	1    6750 3300
 	-1   0    0    1
@@
 F 2 "Connector_PinHeader_2.54mm:PinHeader_2x13_P2.54mm_Horizontal" H 9150 2950 50  0001 C CNN
 F 3 "~" H 9150 2950 50  0001 C CNN
+F 4 "23-0877602616-ND" H 9150 2950 50  0001 C CNN "Digi-Key_PN"
+F 5 "0877602616" H 9150 2950 50  0001 C CNN "MPN"
+F 6 "Molex" H 9150 2950 50  0001 C CNN "Manufacturer"
 	1    9150 2950
 	1    0    0    -1

Commit message: hardware_v3: also add package, description, notes fields for BOM
Parts:
- J1: Description (none) -> 2x1 male header; Notes (none) -> Install J1 jumper to defeat EEPROM write protect; Package (none) -> through-hole (2.54mm pitch)
- J2: Description (none) -> 20x2 female header; Notes (none) -> pi GPIO header; Package (none) -> through-hole (2.54mm pitch)
- J3: Description (none) -> 13x2 male header 90 degree; Notes (none) -> Straight or 90 degree depending on application; Package (none) -> through-hole (2.54mm pitch)
- R2: Description (none) -> 10K, 1/8 watt resistor; Notes (none) -> Pull-up for EEPROM write protect; Package (none) -> 0805
- R3, R4: Description (none) -> 3.9K, 1/8 watt resistor; Notes (none) -> Pull-ups for ID EEPROM; Package (none) -> 0805
- R5: Description (none) -> 1.4K ohm, 1/8 watt resistor; Notes (none) -> Pull-up for STATUS3; Package (none) -> 0805
- U1: Description (none) -> I2C Serial EEPROM 32Kb; Notes (none) -> ID EEPROM; Package (none) -> 8-SOIC
- U2: Description (none) -> 19-bit bus interface with 3-state outputs; Notes (none) -> pin 1 marking oriented opposite J3; Package (none) -> 48-SSOP
Changed lines of the file:
@@
 F 5 "NPPN202AFCN-RC" H 2400 2000 50  0001 C CNN "MPN"
 F 6 "Sullins Connector Solutions" H 2400 2000 50  0001 C CNN "Manufacturer"
+F 7 "through-hole (2.54mm pitch)" H 2400 2000 50  0001 C CNN "Package"
+F 8 "20x2 female header" H 2400 2000 50  0001 C CNN "Description"
+F 9 "pi GPIO header" H 2400 2000 50  0001 C CNN "Notes"
 	1    2400 2000
 	1    0    0    -1
@@
 F 5 "CAT24C32WI-GT3" H 3050 5950 50  0001 C CNN "MPN"
 F 6 "ON Semiconductor" H 3050 5950 50  0001 C CNN "Manufacturer"
+F 7 "8-SOIC" H 3050 5950 50  0001 C CNN "Package"
+F 8 "I2C Serial EEPROM 32Kb" H 3050 5950 50  0001 C CNN "Description"
+F 9 "ID EEPROM" H 3050 5950 50  0001 C CNN "Notes"
 	1    3050 5950
 	1    0    0    -1
@@
 F 5 "ERJ-6ENF3901V" V 3700 5700 50  0001 C CNN "MPN"
 F 6 "Panasonic Electronic Components" V 3700 5700 50  0001 C CNN "Manufacturer"
+F 7 "0805" V 3700 5700 50  0001 C CNN "Package"
+F 8 "3.9K, 1/8 watt resistor" V 3700 5700 50  0001 C CNN "Description"
+F 9 "Pull-ups for ID EEPROM" V 3700 5700 50  0001 C CNN "Notes"
 	1    3700 5700
 	1    0    0    -1
@@
 F 5 "ERJ-6ENF3901V" V 3900 5700 50  0001 C CNN "MPN"
 F 6 "Panasonic Electronic Components" V 3900 5700 50  0001 C CNN "Manufacturer"
+F 7 "0805" V 3900 5700 50  0001 C CNN "Package"
+F 8 "3.9K, 1/8 watt resistor" V 3900 5700 50  0001 C CNN "Description"
+F 9 "Pull-ups for ID EEPROM" V 3900 5700 50  0001 C CNN "Notes"
 	1    3900 5700
 	1    0    0    -1
@@
 F 5 "M20-9990246" H 1500 6200 50  0001 C CNN "MPN"
 F 6 "Harwin Inc." H 1500 6200 50  0001 C CNN "Manufacturer"
+F 7 "through-hole (2.54mm pitch)" H 1500 6200 50  0001 C CNN "Package"
+F 8 "2x1 male header" H 1500 6200 50  0001 C CNN "Description"
+F 9 "Install J1 jumper to defeat EEPROM write protect" H 1500 6200 50  0001 C CNN "Notes"
 	1    1500 6200
 	-1   0    0    1
@@
 F 5 "ERJ-6ENF1002V" V 1850 5700 50  0001 C CNN "MPN"
 F 6 "Panasonic Electronic Components" V 1850 5700 50  0001 C CNN "Manufacturer"
+F 7 "0805" V 1850 5700 50  0001 C CNN "Package"
+F 8 "10K, 1/8 watt resistor" V 1850 5700 50  0001 C CNN "Description"
+F 9 "Pull-up for EEPROM write protect" V 1850 5700 50  0001 C CNN "Notes"
 	1    1850 5700
 	-1   0    0    1
@@
 F 5 "SN74LVC161284DLR" H 7800 2550 50  0001 C CNN "MPN"
 F 6 "Texas Instruments" H 7800 2550 50  0001 C CNN "Manufacturer"
+F 7 "48-SSOP" H 7800 2550 50  0001 C CNN "Package"
+F 8 "19-bit bus interface with 3-state outputs" H 7800 2550 50  0001 C CNN "Description"
+F 9 "pin 1 marking oriented opposite J3" H 7800 2550 50  0001 C CNN "Notes"
 	1    7800 2550
 	1    0    0    -1
@@
 F 5 "ERJ-6ENF1401V" V 6750 3300 50  0001 C CNN "MPN"
 F 6 "Panasonic Electronic Components" V 6750 3300 50  0001 C CNN "Manufacturer"
+F 7 "0805" V 6750 3300 50  0001 C CNN "Package"
+F 8 "1.4K ohm, 1/8 watt resistor" V 6750 3300 50  0001 C CNN "Description"
+F 9 "Pull-up for STATUS3" V 6750 3300 50  0001 C CNN "Notes"
 	1    6750 3300
 	-1   0    0    1
@@
 F 5 "0877602616" H 9150 2950 50  0001 C CNN "MPN"
 F 6 "Molex" H 9150 2950 50  0001 C CNN "Manufacturer"
+F 7 "through-hole (2.54mm pitch)" H 9150 2950 50  0001 C CNN "Package"
+F 8 "13x2 male header 90 degree" H 9150 2950 50  0001 C CNN "Description"
+F 9 "Straight or 90 degree depending on application" H 9150 2950 50  0001 C CNN "Notes"
 	1    9150 2950
 	1    0    0    -1
