File: hardware/v4/pi-parport.sch (KiCad schematic (older format))
At the start: 16 parts, among them J1 CONN_01X02, J2 40HAT, J3 Conn_02x13_Odd_Even, U1 CAT24C32, U2 SN74LVC161284DLR

Commit message: hardware: BOM improvements/fixes.
* Fix capacitor quantity in v4.

* SN74LVC161284DLR Digi-Key part number: cut tape packaging
  discontinued at Digi-Key, use tube packaging instead.

* Fix 40-pin and 26-pin headers, accidentally picked 2 mm pitch parts
  instead of 2.54 mm pitch parts.
Parts:
- J2: Digi-Key_PN S5750-20-ND -> S7123-ND; MPN NPPN202AFCN-RC -> PPPC202LFBN-RC
- J3: Digi-Key_PN 23-0877602616-ND -> 609-3349-ND; MPN 0877602616 -> 68021-226HLF; Manufacturer Molex -> Amphenol ICC (FCI)
- U2: Digi-Key_PN 296-8467-1-ND -> 296-8467-5-ND; MPN SN74LVC161284DLR -> SN74LVC161284DL
Changed lines of the file:
@@
 F 2 "Connector_PinSocket_2.54mm:PinSocket_2x20_P2.54mm_Vertical" H 2400 2200 50  0001 C CNN
 F 3 "" H 1700 2000 50  0000 C CNN
-F 4 "S5750-20-ND" H 2400 2000 50  0001 C CNN "Digi-Key_PN"
-F 5 "NPPN202AFCN-RC" H 2400 2000 50  0001 C CNN "MPN"
+F 4 "S7123-ND" H 2400 2000 50  0001 C CNN "Digi-Key_PN"
+F 5 "PPPC202LFBN-RC" H 2400 2000 50  0001 C CNN "MPN"
 F 6 "Sullins Connector Solutions" H 2400 2000 50  0001 C CNN "Manufacturer"
 F 7 "through-hole (2.54mm pitch)" H 2400 2000 50  0001 C CNN "Package"
@@
 F 2 "Package_SO:SSOP-48_7.5x15.9mm_P0.635mm" H 6700 3000 60  0001 C CNN
 F 3 "http://www.ti.com/lit/ds/symlink/sn74lvc161284.pdf" H 5975 3681 60  0001 C CNN
-F 4 "296-8467-1-ND" H 7800 2550 50  0001 C CNN "Digi-Key_PN"
-F 5 "SN74LVC161284DLR" H 7800 2550 50  0001 C CNN "MPN"
+F 4 "296-8467-5-ND" H 7800 2550 50  0001 C CNN "Digi-Key_PN"
+F 5 "SN74LVC161284DL" H 7800 2550 50  0001 C CNN "MPN"
 F 6 "Texas Instruments" H 7800 2550 50  0001 C CNN "Manufacturer"
 F 7 "48-SSOP" H 7800 2550 50  0001 C CNN "Package"
@@
 F 2 "Connector_PinHeader_2.54mm:PinHeader_2x13_P2.54mm_Horizontal" H 9150 2950 50  0001 C CNN
 F 3 "~" H 9150 2950 50  0001 C CNN
-F 4 "23-0877602616-ND" H 9150 2950 50  0001 C CNN "Digi-Key_PN"
-F 5 "0877602616" H 9150 2950 50  0001 C CNN "MPN"
-F 6 "Molex" H 9150 2950 50  0001 C CNN "Manufacturer"
+F 4 "609-3349-ND" H 9150 2950 50  0001 C CNN "Digi-Key_PN"
+F 5 "68021-226HLF" H 9150 2950 50  0001 C CNN "MPN"
+F 6 "Amphenol ICC (FCI)" H 9150 2950 50  0001 C CNN "Manufacturer"
 F 7 "through-hole (2.54mm pitch)" H 9150 2950 50  0001 C CNN "Package"
 F 8 "13x2 male header 90 degree" H 9150 2950 50  0001 C CNN "Description"
