File: hardware/v5/hat.kicad_sch (KiCad schematic)
At the start: 6 parts, among them J1 GPIO, U1 CAT24C256

Commit message: v5: update page settings
Problem: template pages are A4 size and have have boiler plate
metadata.

Switch to U.S. letter size and update page metadata with project
specific info.
Other:
- company: (none) -> WorlickWerx
- title: (none) -> Pi Parallel Port HAT+
Changed lines of the file:
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@@
 	(generator "eeschema")
 	(generator_version "8.0")
-	(paper "A4")
+	(paper "USLetter")
 	(title_block
-		(date "15 nov 2012")
+		(title "Pi Parallel Port HAT+")
+		(date "2024-08-25")
+		(rev "v5")
+		(company "WorlickWerx")
+		(comment 1 "CERN-OHL-1.2")
 	)
 	(junction
